Commit message: feat: updates to current state of development which completely removes need for gazebo

File: src/robot_description/rb_theron_common/rb_theron_description/robots/rb_theron.urdf.xacro (robot description, xacro)
@@ -28,18 +28,146 @@
 	<xacro:arg name="prefix" default=""/>
 	<!-- <xacro:arg name="gpu" default="true"/> -->
+	<!-- ros2_control_hardware_type:
+		mock_components = ros2_control only in rviz
+		gz_ros2_control = ros2_control in gazebo
+		dryve_d1 = ros2_control only in real life
+	-->
+    <xacro:arg name="ros2_control_hardware_type" default="mock_components" />
+	<xacro:arg name="ros_distro" default="humble" />
 	<!-- *************** -->
 	<!-- Robots Elements -->
 	<!-- *************** -->
 	<!-- base with wheels -->
-	<xacro:rb_theron_base prefix="$(arg prefix)" hq="${hq}" publish_bf="${publish_bf}" />
+	<xacro:rb_theron_base
+	  prefix="$(arg prefix)"
+	  hq="${hq}"
+	  publish_bf="${publish_bf}"
+	  ros2_control_hardware_type="$(arg ros2_control_hardware_type)"
+	  ros_distro="$(arg ros_distro)">
+	</xacro:rb_theron_base>
 	<!-- Gazebo ros control pluggins -->
 	<!-- <xacro:ros_control/> -->
 	<xacro:gazebo_colors prefix="$(arg prefix)"/>
+	<!-- SENSORS  DEBUGG-->
+	<!-- TODO: Should be sensor_intel_d435, but this one isn't migrated to ros2 yet -->
+	<!-- TODO: Moved 0.01 in x, otherwise the camera is still inside the robot -->
+	<xacro:sensor_r430 prefix="$(arg prefix)front_realsense_camera" parent="$(arg prefix)base_link" publish_bf="${publish_bf}" robot_name="${robot_name}" prefix_topic="front_realsense_camera" hq="${hq}">
+		<origin xyz="0.3305 0.0 0.1468" rpy="0 0 0"/>
+	</xacro:sensor_r430>
+	<xacro:sensor_r430 prefix="$(arg prefix)back_realsense_camera" parent="$(arg prefix)base_link" publish_bf="${publish_bf}" robot_name="${robot_name}" prefix_topic="back_realsense_camera" hq="${hq}">
+		<origin xyz="-0.3305 0.0 0.1468" rpy="0 0 3.1416"/>
+	</xacro:sensor_r430>
+	<!--Added back top realsense camera because running YOLO network on depthai camera in simulation reduces Real Time Factor (RTF)-->
+	<xacro:sensor_r430 prefix="$(arg prefix)back_top_realsense_camera" parent="$(arg prefix)base_link" publish_bf="${publish_bf}" robot_name="${robot_name}" prefix_topic="back_top_realsense_camera" hq="${hq}">
+		<origin xyz="-0.3305 0.0 1.1468" rpy="0 0 3.1416"/>
+	</xacro:sensor_r430>
+	<!-- TODO: Moved 0.01 in x, otherwise the camera is still inside the robot -->
+	<!--xacro:sensor_orbbec_astra prefix="$(arg prefix)front_rgbd_camera" parent="$(arg prefix)base_link" prefix_topic="front_rgbd_camera">
+		<origin xyz="0.3305 0.0 0.1898" rpy="0 0 0"/>
+	</xacro:sensor_orbbec_astra -->
+	<xacro:sensor_imu_hector prefix="$(arg prefix)imu" parent="$(arg prefix)base_link">
+		<origin xyz="-0.1975 0.0 0.1598" rpy="0 0 0"/>
+	</xacro:sensor_imu_hector>
+	<xacro:sensor_sick_nanoscan3 prefix="$(arg prefix)front_laser" parent="$(arg prefix)base_link" publish_bf="${publish_bf}" robot_name="${robot_name}" prefix_topic="front_laser" hq="${hq}" min_angle="-1.9507619" max_angle="1.9507619" gpu="true">
+		<origin xyz="0.250 0.0 0.1643" rpy="0 3.1416 3.1416"/>
+	</xacro:sensor_sick_nanoscan3>
+	<!--<xacro:sensor_rs_lidar_16 prefix="$(arg prefix)top_laser" parent="$(arg prefix)base_link" prefix_topic="top_laser" min_angle="-3.1416" max_angle="3.1416">
+		<origin xyz="0.214 0.0 0.275" rpy="-1.57079632679 0 -0.23"/>
+	</xacro:sensor_rs_lidar_16>-->
+	<xacro:sensor_rs_bpearl prefix="$(arg prefix)top_laser" parent="$(arg prefix)base_link" publish_bf="${publish_bf}" robot_name="${robot_name}" prefix_topic="top_laser" hq="${hq}" range_min="0.1" range_max="90" hfov="360" samples="1800" vfov="90.0" lasers="32" fps="10" gpu="false">
+		<origin xyz="0.3 -0.175 1.165" rpy="-1.570796326795 0 -1.570796326795"/>
+		<!-- positions of the b-pearl based on solid: xyz="0.333 -0.180 1.194" rpy="-1.570796326795 0 -1.570796326795" -->
+	</xacro:sensor_rs_bpearl>
+	<!-- <xacro:sensor_sick_nanoscan3 prefix="$(arg prefix)back_laser" parent="$(arg prefix)base_link" prefix_topic="back_laser" min_angle="-1.8107619" max_angle="1.8107619">
+		<origin xyz="-0.250 0.0 0.1643" rpy="0 3.1416 0"/>
+	</xacro:sensor_sick_nanoscan3> -->
+	<xacro:arg name="front_oak_d_camera_model" default="OAK-D-S2" />
+	<xacro:arg name="front_oak_d_base_frame" default="oak-d-s2-usb-base--frame" />
+	<xacro:arg name="front_oak_d_pos_x" default="0.317" />
+	<xacro:arg name="front_oak_d_pos_y" default="-0.197" />
+	<xacro:arg name="front_oak_d_pos_z" default="1.3044" />
+	<xacro:arg name="front_oak_d_roll" default="0.0" />
+	<xacro:arg name="front_oak_d_pitch" default="0.0" />
+	<xacro:arg name="front_oak_d_yaw" default="0.0" />
+	<xacro:depthai_camera
+		prefix="$(arg prefix)front_top_oak_d_camera"
+		parent="$(arg prefix)base_link"
+		publish_bf="${publish_bf}"
+		robot_name="${robot_name}"
+		prefix_topic="front_top_oak_d_camera"
+		camera_model="$(arg front_oak_d_camera_model)"
+		base_frame="$(arg front_oak_d_base_frame)"
+		cam_pos_x="$(arg front_oak_d_pos_x)"
+		cam_pos_y="$(arg front_oak_d_pos_y)"
+		cam_pos_z="$(arg front_oak_d_pos_z)"
+		cam_roll="$(arg front_oak_d_roll)"
+		cam_pitch="$(arg front_oak_d_pitch)"
+		cam_yaw="$(arg front_oak_d_yaw)"
+		hq="${hq}">
+	</xacro:depthai_camera>
+	<!-- ROBAST Module Cage -->
+	<xacro:include filename="$(find rb_theron_description)/urdf/module_cage/module_cage.urdf.xacro" />
+	<xacro:module_cage prefix="$(arg prefix)" parent="$(arg prefix)base_link" hq="${hq}">
+		<origin xyz="-0.15 0.0 0.725" rpy="0 0 0"/>
+	</xacro:module_cage>
+	<!-- ROBAST Drawer -->
+	<xacro:include filename="$(find rb_theron_description)/urdf/drawer/drawer.urdf.xacro" />
+	<xacro:drawer
+	    prefix="$(arg prefix)"
+		suffix="5"
+		parent="$(arg prefix)base_link"
+		ros2_control_hardware_type="$(arg ros2_control_hardware_type)"
+		ros_distro="$(arg ros_distro)"
+		drawer_size_z="0.28">
+		<origin xyz="0.125 0.0 0.42" rpy="0 0 0"/>
+	</xacro:drawer>
+	<xacro:drawer
+	    prefix="$(arg prefix)"
+		suffix="4"
+		parent="$(arg prefix)base_link"
+		ros2_control_hardware_type="$(arg ros2_control_hardware_type)"
+		ros_distro="$(arg ros_distro)"
+		drawer_size_z="0.18">
+		<origin xyz="0.125 0.0 0.67" rpy="0 0 0"/>
+	</xacro:drawer>
+	<xacro:drawer
+	    prefix="$(arg prefix)"
+		suffix="3"
+		parent="$(arg prefix)base_link"
+		ros2_control_hardware_type="$(arg ros2_control_hardware_type)"
+		ros_distro="$(arg ros_distro)"
+		drawer_size_z="0.08">
+		<origin xyz="0.125 0.0 0.82" rpy="0 0 0"/>
+	</xacro:drawer>
+	<xacro:drawer
+		prefix="$(arg prefix)"
+		suffix="2"
+		parent="$(arg prefix)base_link"
+		ros2_control_hardware_type="$(arg ros2_control_hardware_type)"
+		ros_distro="$(arg ros_distro)"
+		drawer_size_z="0.08">
+		<origin xyz="0.125 0.0 0.92" rpy="0 0 0"/>
+	</xacro:drawer>
+	<xacro:drawer
+		prefix="$(arg prefix)"
+		suffix="1"
+		parent="$(arg prefix)base_link"
+		ros2_control_hardware_type="$(arg ros2_control_hardware_type)"
+		ros_distro="$(arg ros_distro)"
+		drawer_size_z="0.08">
+		<origin xyz="0.125 0.0 1.02" rpy="0 0 0"/>
+	</xacro:drawer>
 	<!-- ROBAST Door Opening Mechanism -->
 	<xacro:include filename="$(find rb_theron_description)/urdf/door_opening_mechanism/door_opening_mechanism.urdf.xacro" />
-	<xacro:door_opening_mechanism prefix="$(arg prefix)" parent="$(arg prefix)base_link" hq="${hq}">
+	<xacro:door_opening_mechanism
+	    prefix="$(arg prefix)"
+		parent="$(arg prefix)base_link"
+		ros2_control_hardware_type="$(arg ros2_control_hardware_type)"
+		ros_distro="$(arg ros_distro)"
+		hq="${hq}">
 		<origin xyz="-0.3 0 0.225" rpy="0 0 0"/>
 	</xacro:door_opening_mechanism>
-	<!-- Gazebo ros control pluggins -->
-	<xacro:ros_control prefix="$(arg prefix)" publish_bf="${publish_bf}"/>
+	<!-- Gazebo plugins -->
+	<xacro:ros_control ros_distro="$(arg ros_distro)"/>
+	<xacro:gazebo_sensor_plugins ros_distro="$(arg ros_distro)"/>
 </robot>

File: src/robot_description/rb_theron_common/rb_theron_description/urdf/bases/theron_base.urdf.xacro (robot description, xacro)
@@ -4,5 +4,5 @@
     <inertia  ixx="${m*(y*y+z*z)/12}" ixy = "0" ixz = "0"
               iyy="${m*(x*x+z*z)/12}" iyz = "0"
-              izz="${m*(x*x+z*z)/12}" />
+              izz="${m*(x*x+y*y)/12}" />
   </xacro:macro>
   <xacro:macro name="theron_base" params="prefix publish_bf hq">
@@ -58,5 +58,5 @@
         <origin xyz="0 0 0.105" rpy="0 0 0 " />
         <geometry>
-          <box size="0.390 0.240 0.165"/>
+          <box size="0.390 0.240 0.140"/>
           <!-- <mesh filename="(find rb_theron_description)/meshes/bases/theron_base.dae"/> -->
         </geometry>

File: src/robot_description/rb_theron_common/rb_theron_description/urdf/common.gazebo.xacro (robot description, xacro)
@@ -2,30 +2,33 @@
 <robot xmlns:xacro="http://www.ros.org/wiki/xacro">
     <!-- ROS CONTROL GAZEBO PLUGIN -->
-    <xacro:macro name="ros_control" params="prefix publish_bf">
+    <xacro:macro name="ros_control" params="ros_distro">
         <gazebo>
-            <!-- <plugin filename="libgazebo_ros2_control.so" name="gazebo_ros2_control">
-				<parameters>$(find rb_theron_description)/config/rb_theron_controller.yaml</parameters>
-			</plugin> -->
-            <plugin filename="libgz-sim-joint-state-publisher-system" name="gz::sim::systems::JointStatePublisher">
-            </plugin>
-            <plugin filename="libgz-sim-diff-drive-system.so" name="gz::sim::systems::DiffDrive">
-                <left_joint>$(arg prefix)left_wheel_joint</left_joint>
-                <right_joint>$(arg prefix)right_wheel_joint</right_joint>
-                <wheel_separation>0.5032</wheel_separation>
-                <wheel_radius>0.0762</wheel_radius>
-                <odom_publish_frequency>30</odom_publish_frequency>
-                <topic>cmd_vel</topic>
-                <frame_id>$(arg prefix)odom</frame_id>
-                <!-- There is no possiblity (as far as I know) to disable tf publishing of odom->base, so if you
-				don't want the tf to be published, you can just dump it into a different topic -->
-                <!-- <tf_topic>tf_dump</tf_topic> -->
-                <xacro:if value="${publish_bf}">
-                    <child_frame_id>$(arg prefix)base_footprint</child_frame_id>
-                </xacro:if>
-                <xacro:unless value="${publish_bf}">
-                    <child_frame_id>$(arg prefix)base_link</child_frame_id>
-                </xacro:unless>
-            </plugin>
+            <xacro:if value="${ros_distro == 'humble'}">
+                <plugin name="ign_ros2_control::IgnitionROS2ControlPlugin" filename="libign_ros2_control-system.so">
+                    <parameters>$(find rb_theron_description)/config/rb_theron_gz_ros2_controller.yaml</parameters>
+                </plugin>
+            </xacro:if>
+            <xacro:unless value="${ros_distro == 'humble'}">
+                <plugin name="gz_ros2_control::GazeboSimROS2ControlPlugin" filename="gz_ros2_control-system">
+                    <parameters>$(find rb_theron_description)/config/rb_theron_gz_ros2_controller.yaml</parameters>
+                </plugin>
+            </xacro:unless>
         </gazebo>
+    </xacro:macro>
+    <xacro:macro name="gazebo_sensor_plugins" params="ros_distro">
+        <gazebo>
+            <xacro:if value="${ros_distro == 'humble'}">
+                <plugin name="ignition::gazebo::systems::Imu" filename="libignition-gazebo-imu-system.so"></plugin>
+                <plugin name="ignition::gazebo::systems::Sensors" filename="libignition-gazebo-sensors-system.so">
+                    <render_engine>ogre2</render_engine>
+                </plugin>
+            </xacro:if>
+            <xacro:unless value="${ros_distro == 'humble'}">
+                <plugin name="gz::sim::systems::Imu" filename="libgz-sim-imu-system"></plugin>
+                <plugin name="gz::sim::systems::Sensors" filename="libgz-sim-sensors-system.so">
+                    <render_engine>ogre2</render_engine>
+                </plugin>
+            </xacro:unless>
+		</gazebo>
     </xacro:macro>
     <xacro:macro name="gazebo_colors" params="prefix">
